Commit message: Fix Camera and LIDAR Position

File: racer_ws/src/racer_description/urdf/racer.xacro (robot description, xacro)
@@ -179,5 +179,5 @@
   <joint name="camera_joint" type="fixed">
     <axis xyz="0 1 0" />
-    <origin xyz=".2 0 0.5" rpy="0 0 0"/>
+    <origin xyz=".21 0 0.075" rpy="0 0 0"/>
     <parent link="chassis"/>
     <child link="camera"/>
@@ -185,5 +185,5 @@
   <joint name="hokuyo_joint" type="fixed">
     <axis xyz="0 1 0" />
-    <origin xyz=".15 0 .1" rpy="0 0 0"/>
+    <origin xyz=".21 0 .135" rpy="0 0 0"/>
     <parent link="chassis"/>
     <child link="hokuyo"/>

Commit message: Changed hokuyo parameters and fixed camera position and added cameraIner parameter (not working yet)

File: racer_ws/src/racer_description/urdf/racer.xacro (robot description, xacro)
@@ -6,4 +6,5 @@
   <xacro:property name="cameraSize" value="0.05"/>
   <xacro:property name="cameraMass" value="0.1"/>
+  <xacro:property name="cameraIner" value="(${cameraMass}/12 * (2*(${cameraSize}**2)))"/>
   <!--  body  -->
   <link name='chassis'>
@@ -174,5 +175,5 @@
       <origin xyz="0 0 0" rpy="0 0 0"/>
       <box_inertia m="${cameraMass}" x="${cameraSize}" y="${cameraSize}" z="${cameraSize}" />
-      <inertia ixx="1e-6" ixy="0" ixz="0" iyy="1e-6" iyz="0" izz="1e-6" />
+      <inertia ixx="0.1" ixy="0" ixz="0" iyy="0.1" iyz="0" izz="0.1" />
     </inertial>
   </link>
